File: PCB/DangerDonut.kicad_sch (KiCad schematic)
At the start: 42 parts, among them SW2 SW_Push, SW3 SW_Push, U1 ADXL375BCCZ-RL7, U2 MIC5219-5.0YM5, U3 MIC5219-3.3YM5, U4 TSSP58038, U5 ESP32-S3-WROOM-1-N16

Commit message: updated PCB
Parts:
- removed D12, D13, D14, D15: HD107S, HD107S, symbol HD107S:HD107S
- removed H4: ~, Round_Nut:SMTSO2515, symbol SMD_round_nut:SMTSO2515
- added C10: 10 uF, symbol Device:C
- added C11, C12, C14, C15, C16, C17, C18, C19, C20, C21: 100 nF, symbol Device:C
- added C13: 22 uF, symbol Device:C
- added D12: 1N5819, symbol Device:D
- added D13: Z3.3V, symbol Device:D_Zener
- added J1: ~, TYPEC-300D-BCP16H88:TYPEC-300D-BCP16H88, symbol TYPEC-300D-BCP16H88:TYPEC-300D-BCP16H88
- added J2, J3: ~, ESC_XSD7A:ESC_XSD7A, symbol ESC XSD7A:ESC_XSD7A
- added R10, R7, R9: 100, symbol Device:R
- added R11: 10k, symbol Device:R
- added R12, R5, R6: 5.1K, symbol Device:R
- added R13: 1.5K, symbol Device:R
- added R8: 68, symbol Device:R
- C6, C8, C9: value 0.1 uF -> 100 nF
Connections:
- net +3.3V: now also R11.1
- net +3V3: now also U1.1 (VDDI/O), C12.2, R7.2, R8.1
- net +5V: now also C15.2, C16.2, C17.2, C18.2, C19.2, C20.2
- net +BATT: now also C13.1, C14.1, D12.1 (K), J2.4 (Vcc), J3.4 (Vcc), R12.1
- net GND: now also C9.2, C10.2, C11.2, C12.1, C13.2, C14.2, C15.1, C16.1, C17.1, C18.1, C19.1, C20.1, C21.2, D13.2 (A), J1.1 (Shell), J1.A1 (GND), J1.A12 (GND), J1.B1 (GND), J1.B12 (GND), J2.1 (GND), J2.2 (D_GND), J3.1 (GND), J3.2 (D_GND), R13.2, R5.2, R6.2
- net D5_CO: now reaches D5.2 (CO), D6.5 (CI)
- net D5_DO: now reaches D5.3 (DO), D6.6 (DI)
- net at C6.1, R4.2, SW2.1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: no longer C9.2
- net Accel_DO: now reaches U1.12 (SDO/ALTADDRESS)
- net Accel_DI: now reaches U1.13 (SDA/SDI/SDIO)
- net Accel_clock: now reaches U1.14 (SCL/SCLK)
- net at U1.6 (VS): now also C10.1, C11.1, R8.2
- net Accel_CS: now reaches U1.7 (*CS)
- net Accel_CS: now also R11.2
- net Accel_INT1: now reaches U1.8 (INT1)
- net Accel_INT2: now reaches U1.9 (INT2)
- net at D10.2 (CO): no longer D11.5 (CI)
- net at D10.3 (DO): no longer D11.6 (DI)
- net IR_out: now reaches U4.1 (OUT)
- net at U4.3 (Vs): now also C9.1, R7.1
- net D-: now reaches U5.13 (IO19)
- net D-: now also J1.A7 (D-), J1.B7 (D-)
- net D+: now reaches U5.14 (IO20)
- net D+: now also J1.A6 (D+), J1.B6 (D+)
- net LED_clock: now reaches D1.5 (CI)
- net LED_clock: now also D11.5 (CI)
- net LED_data: now reaches D1.6 (DI)
- net LED_data: now also D11.6 (DI)
- net BOOT: no longer names the net of SW3.2, U5.27 (IO0)
- net BOOT: no longer C9.1
- net D7 CO: no longer names the net of D7.2 (CO), D8.5 (CI)
- net D7 DO: no longer names the net of D7.3 (DO), D8.6 (DI)
- net EN: no longer names the net of C5.1, C6.2, R3.1, SW2.2, U5.3 (EN)
- new net: J2.3 (Data), R9.1
- new net: J1.A5 (CC1), R5.1
- new net: D12.2 (A), J1.A4 (VBUS), J1.A9 (VBUS), J1.B4 (VBUS), J1.B9 (VBUS)
- new net: J1.B5 (CC2), R6.1
- new net: J3.3 (Data), R10.1
- new net BATT: C21.1, D13.1 (K), R12.2, R13.1
- new net ESC_data_L: R9.2
- new net ESC_data_R: R10.2
Other:
- note removed: "TODO: USB Port USB power diodes Hookup ESP32 TSSP58038 ADXL375 ESC output pads"
- title: Danger Cookie -> Danger Donut
- moved on the sheet: BT1, BT2, C1, C2, C3, C4, C5, C6, C7, C8, D1, D10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
